Commit message: i controller added, before invkintraj

File: RobotSystem/RobotModel/Robot/Draco/DracoFixedNoVisualDrake.urdf (robot description, URDF)
Before this commit: robot Draco, 17 links, 16 joints
Links:
- removed link basePosX
- removed link basePosY
- removed link basePosZ
- removed link baseRotY
- removed link baseRotZ
- removed link world
- link lAnkle: geometry collision box size=0.15 0.04 0.03
- link lHipPitch: geometry 
- link lHipRoll: geometry 
- link lHipYaw: geometry 
- link lKnee: geometry 
- link rAnkle: geometry collision box size=0.15 0.04 0.03
- link rHipPitch: geometry 
- link rHipRoll: geometry 
- link rHipYaw: geometry 
- link rKnee: geometry 
Joints:
- removed joint basePosX
- removed joint basePosY
- removed joint basePosZ
- removed joint baseRotX
- removed joint baseRotY
- removed joint baseRotZ
