Commit message: under onstep planning

File: RobotSystem/RobotModel/Robot/Draco/DracoDebug.urdf (robot description, URDF)
Before this commit: robot Draco, 17 links, 16 joints
Links:
- removed link basePosX
- removed link basePosY
- removed link basePosZ
- removed link baseRotY
- removed link baseRotZ
Joints:
- removed joint basePosX
- removed joint basePosY
- removed joint basePosZ
- removed joint baseRotY
- removed joint baseRotZ
- joint baseRotX: axis 1 0 0 -> (none); parent baseRotY -> world; type continuous -> floating
- joint lAnkle: limit lower=0.901 upper=2.44 effort=40 velocity=25.0 -> (none); type revolute -> continuous
- joint lHipPitch: limit lower=-1.04 upper=1.04 effort=40 velocity=25.0 -> (none); type revolute -> continuous
- joint lHipRoll: limit lower=-0.52 upper=1.04 effort=40 velocity=25.0 -> (none); type revolute -> continuous
- joint lHipYaw: limit lower=-1.04 upper=1.04 effort=40 velocity=25.0 -> (none); type revolute -> continuous
- joint lKnee: limit lower=0.0 upper=2.13 effort=40 velocity=25.0 -> (none); type revolute -> continuous
- joint rAnkle: limit lower=0.901 upper=2.44 effort=40 velocity=25.0 -> (none); type revolute -> continuous
- joint rHipPitch: limit lower=-1.04 upper=1.04 effort=40 velocity=25.0 -> (none); type revolute -> continuous
- joint rHipRoll: limit lower=-1.04 upper=0.52 effort=40 velocity=25.0 -> (none); type revolute -> continuous
- joint rHipYaw: limit lower=-1.04 upper=1.04 effort=40 velocity=25.0 -> (none); type revolute -> continuous
- joint rKnee: limit lower=0.0 upper=2.13 effort=40 velocity=25.0 -> (none); type revolute -> continuous

Commit message: sync

File: RobotSystem/RobotModel/Robot/Draco/DracoDebug.urdf (robot description, URDF)
Before this commit: robot Draco, 12 links, 11 joints
Links:
- link lAnkle: geometry visual mesh filename=meshes/lAnkle.dae
