Commit message: fixed draco added

File: RobotSystem/RobotModel/Robot/Draco/DracoFixed.urdf (robot description, URDF)
Before this commit: robot Draco, 11 links, 10 joints
Links:
- added link world, mass 0.00000001
- link torso: geometry visual mesh filename=meshes/torso_.dae
Joints:
- added joint torso: type fixed, parent world, child torso, origin xyz=0 0 1.5 rpy=0 0 0

Commit message: joint test added

File: RobotSystem/RobotModel/Robot/Draco/DracoFixed.urdf (robot description, URDF)
Before this commit: robot FixedDraco, 12 links, 11 joints
Joints:
- joint lAnkle: limit lower=0.901 upper=2.44 effort=40 velocity=25.0 -> (none); type revolute -> continuous
- joint lHipPitch: limit lower=-1.04 upper=1.04 effort=40 velocity=25.0 -> (none); type revolute -> continuous
- joint lHipRoll: limit lower=-0.52 upper=1.04 effort=40 velocity=25.0 -> (none); type revolute -> continuous
- joint lHipYaw: limit lower=-1.04 upper=1.04 effort=40 velocity=25.0 -> (none); type revolute -> continuous
- joint lKnee: limit lower=0.0 upper=2.13 effort=40 velocity=25.0 -> (none); type revolute -> continuous
- joint rAnkle: limit lower=0.901 upper=2.44 effort=40 velocity=25.0 -> (none); type revolute -> continuous
- joint rHipPitch: limit lower=-1.04 upper=1.04 effort=40 velocity=25.0 -> (none); type revolute -> continuous
- joint rHipRoll: limit lower=-1.04 upper=0.52 effort=40 velocity=25.0 -> (none); type revolute -> continuous
- joint rHipYaw: limit lower=-1.04 upper=1.04 effort=40 velocity=25.0 -> (none); type revolute -> continuous
- joint rKnee: limit lower=0.0 upper=2.13 effort=40 velocity=25.0 -> (none); type revolute -> continuous

Commit message: sync

File: RobotSystem/RobotModel/Robot/Draco/DracoFixed.urdf (robot description, URDF)
Before this commit: robot FixedDraco, 12 links, 11 joints
Links:
- link lHipPitch: mass 5.5 -> 5.0
- link lKnee: mass 3.0 -> 3.1
- link rHipPitch: mass 6.0 -> 5.0
- link rKnee: mass 3.5 -> 3.1
