Commit message: draco visualization done

File: RobotSystem/RobotModel/Robot/Draco/Draco.urdf (robot description, URDF)
Before this commit: robot Draco, 11 links, 10 joints
Links:
- added link world
- link torso: geometry visual mesh filename=meshes/torso.STL
Joints:
- added joint ground_joint: type floating, parent world, child torso, origin xyz=0 0 0 rpy=0 0 0
- joint lAnkle: origin xyz=0.00107750129935319 0.0167500014015612 -0.480000014901359 rpy=1.92592994438724E-34 0 0 -> xyz=0.00107750129935319 0.0167500014015612 -0.480000014901359 rpy=0 -1.57 0
- joint rAnkle: origin xyz=0.0010775 -0.01675 -0.48 rpy=1.9259E-34 0 0 -> xyz=0.0010775 -0.01675 -0.48 rpy=0 -1.57 0
- joint rKnee: origin xyz=0 0.01675 -0.48 rpy=1.9259E-34 0 0 -> xyz=0 0.01675 -0.48 rpy=0 0 0

Commit message: under wbc debugging

File: RobotSystem/RobotModel/Robot/Draco/Draco.urdf (robot description, URDF)
Before this commit: robot Draco, 12 links, 11 joints
Links:
- link lAnkle: geometry collision box size=0.15 0.04 0.03; visual mesh filename=meshes/lAnkle.dae
- link rAnkle: geometry collision box size=0.15 0.04 0.03; visual mesh filename=meshes/rAnkle.dae
- link torso: geometry 

Commit message: joint position task working

File: RobotSystem/RobotModel/Robot/Draco/Draco.urdf (robot description, URDF)
Before this commit: robot Draco, 12 links, 11 joints
Links:
- link lAnkle: mass 0.308587643244722 -> 0.5
- link lHipPitch: mass 3.50208712499242 -> 6.0
- link lHipRoll: mass 0.357278398824283 -> 0.5
- link lHipYaw: mass 0.892151245856688 -> 1.0
- link lKnee: mass 1.92207078647823 -> 3.8
- link rAnkle: mass 0.308587643109314 -> 0.5
- link rHipPitch: mass 3.50208703325148 -> 6.0
- link rHipRoll: mass 0.357278415264791 -> 0.5
- link rHipYaw: mass 0.89215124347132 -> 1.0
- link rKnee: mass 1.92207077376842 -> 3.8
- link torso: mass 6.20812004330114 -> 12.0

Commit message: make ubuntu work

File: RobotSystem/RobotModel/Robot/Draco/Draco.urdf (robot description, URDF)
Before this commit: robot Draco, 12 links, 11 joints
Joints:
- joint lAnkle: limit lower=0.901 upper=2.44 -> (none); type revolute -> continuous
- joint lHipPitch: type revolute -> continuous
- joint lHipRoll: type revolute -> continuous
- joint lHipYaw: type revolute -> continuous
- joint lKnee: limit lower=0.0 upper=2.13 -> (none); type revolute -> continuous
- joint rAnkle: limit lower=0.901 upper=2.44 -> (none); type revolute -> continuous
- joint rHipPitch: type revolute -> continuous
- joint rHipRoll: type revolute -> continuous
- joint rHipYaw: type revolute -> continuous
- joint rKnee: limit lower=0.0 upper=2.13 -> (none); type revolute -> continuous

Commit message: floating draco mathmatica added

File: RobotSystem/RobotModel/Robot/Draco/Draco.urdf (robot description, URDF)
Before this commit: robot Draco, 12 links, 11 joints
Links:
- added link basePosX
- added link basePosY
- added link basePosZ
- added link baseRotY
- added link baseRotZ
- link torso: geometry 
Joints:
- removed joint ground_joint
- added joint basePosX: type prismatic, parent world, child basePosX, origin xyz=0 0 0 rpy=0 0 0, axis 1 0 0, limit lower=-200. upper=200. effort=100.0 velocity=100.0
- added joint basePosY: type prismatic, parent basePosX, child basePosY, origin xyz=0 0 0 rpy=0 0 0, axis 0 1 0, limit lower=-200. upper=200. effort=100.0 velocity=100.0
- added joint basePosZ: type prismatic, parent basePosY, child basePosZ, origin xyz=0 0 0 rpy=0 0 0, axis 0 0 1, limit lower=-200. upper=200. effort=100.0 velocity=100.0
- added joint baseRotX: type continuous, parent baseRotY, child torso, origin xyz=0 0 0 rpy=0 0 0, axis 1 0 0
- added joint baseRotY: type continuous, parent baseRotZ, child baseRotY, origin xyz=0 0 0 rpy=0 0 0, axis 0 1 0
- added joint baseRotZ: type continuous, parent basePosZ, child baseRotZ, origin xyz=0 0 0 rpy=0 0 0, axis 0 0 1

Commit message: unittest for mathematica functions for model

File: RobotSystem/RobotModel/Robot/Draco/Draco.urdf (robot description, URDF)
Before this commit: robot Draco, 17 links, 16 joints
Links:
- link basePosX: mass None -> 0.0
- link basePosY: mass None -> 0.0
- link basePosZ: mass None -> 0.0
- link baseRotY: mass None -> 0.0
- link baseRotZ: mass None -> 0.0
- link world: mass None -> 0.0

Commit message: new urdf

File: RobotSystem/RobotModel/Robot/Draco/Draco.urdf (robot description, URDF)
Before this commit: robot Draco, 17 links, 16 joints
Links:
- link basePosX: mass 0.0 -> 0.00000001
- link basePosY: mass 0.0 -> 0.00000001
- link basePosZ: mass 0.0 -> 0.00000001
- link baseRotY: mass 0.0 -> 0.00000001
- link baseRotZ: mass 0.0 -> 0.00000001
- link lAnkle: mass 0.5 -> 0.7
- link lHipRoll: mass 0.5 -> 0.408
- link lHipYaw: mass 1.0 -> 2.962
- link lKnee: mass 3.8 -> 3.5
- link rAnkle: mass 0.5 -> 0.7
- link rHipRoll: mass 0.5 -> 0.408
- link rHipYaw: mass 1.0 -> 2.962
- link rKnee: mass 3.8 -> 3.5
- link torso: mass 12.0 -> 9.67; geometry visual mesh filename=meshes/torso.dae
- link world: mass 0.0 -> 0.00000001
Joints:
- joint lAnkle: limit (none) -> lower=0.901 upper=2.44 effort=40 velocity=25.0; origin xyz=0.00107750129935319 0.0167500014015612 -0.480000014901359 rpy=0 -1.57 0 -> xyz=0.0011 0.0168 -0.48 rpy=0 -1.57 0; type continuous -> revolute
- joint lHipPitch: limit (none) -> lower=-1.04 upper=1.04 effort=40 velocity=25.0; origin xyz=0 0.0099999999999999 -0.065 rpy=0 0 0 -> xyz=0 0.010 -0.065 rpy=0 0 0; type continuous -> revolute
- joint lHipRoll: limit (none) -> lower=-0.52 upper=1.04 effort=40 velocity=25.0; origin xyz=0 0.0699999999999993 -0.0200000000000001 rpy=1.92592994438724E-34 0 0 -> xyz=0 0.07 -0.02 rpy=0 0 0; type continuous -> revolute
- joint lHipYaw: limit (none) -> lower=-1.04 upper=1.04 effort=40 velocity=25.0; origin xyz=-0.0222250000000002 0.0870035316828367 -0.29508 rpy=1.92592994438724E-34 0 0 -> xyz=-0.0222 0.0870 -0.2951 rpy=0 0 0; type continuous -> revolute
- joint lKnee: limit (none) -> lower=0.0 upper=2.13 effort=40 velocity=25.0; origin xyz=0 -0.016750000238715 -0.48 rpy=1.92592994438724E-34 0 0 -> xyz=0 -0.0168 -0.48 rpy=0 0 0; type continuous -> revolute
- joint rAnkle: limit (none) -> lower=0.901 upper=2.44 effort=40 velocity=25.0; origin xyz=0.0010775 -0.01675 -0.48 rpy=0 -1.57 0 -> xyz=0.0011 -0.0168 -0.48 rpy=0 -1.57 0; type continuous -> revolute
- joint rHipPitch: limit (none) -> lower=-1.04 upper=1.04 effort=40 velocity=25.0; origin xyz=0 -0.01 -0.065 rpy=1.9259E-34 0 0 -> xyz=0 -0.01 -0.065 rpy=0 0 0; type continuous -> revolute
- joint rHipRoll: limit (none) -> lower=-1.04 upper=0.52 effort=40 velocity=25.0; origin xyz=0 -0.07 -0.02 rpy=1.9259E-34 0 0 -> xyz=0 -0.07 -0.02 rpy=0 0 0; type continuous -> revolute
- joint rHipYaw: limit (none) -> lower=-1.04 upper=1.04 effort=40 velocity=25.0; origin xyz=-0.022225 -0.086996 -0.29508 rpy=1.9259E-34 0 0 -> xyz=-0.0222 -0.0870 -0.2951 rpy=0 0 0; type continuous -> revolute
- joint rKnee: limit (none) -> lower=0.0 upper=2.13 effort=40 velocity=25.0; type continuous -> revolute

File: RobotSystem/RobotModel/Robot/Draco/DracoFixed.urdf (robot description, URDF)
Before this commit: robot DracoFixed, 12 links, 11 joints
Links:
- removed link world
- link lAnkle: mass 0.5 -> 0.7
- link lHipRoll: mass 0.5 -> 0.408
- link lHipYaw: mass 1.0 -> 2.962
- link lKnee: mass 3.8 -> 3.5
- link rAnkle: mass 0.5 -> 0.7
- link rHipRoll: mass 0.5 -> 0.408
- link rHipYaw: mass 1.0 -> 2.962
- link rKnee: mass 3.8 -> 3.5
- link torso: mass 12.0 -> 9.67; geometry visual mesh filename=meshes/torso.dae
Joints:
- removed joint ground_joint
- joint lAnkle: limit (none) -> lower=0.901 upper=2.44 effort=40 velocity=25.0; origin xyz=0.00107750129935319 0.0167500014015612 -0.480000014901359 rpy=0 -1.57 0 -> xyz=0.0011 0.0168 -0.48 rpy=0 -1.57 0; type continuous -> revolute
- joint lHipPitch: limit (none) -> lower=-1.04 upper=1.04 effort=40 velocity=25.0; origin xyz=0 0.0099999999999999 -0.065 rpy=0 0 0 -> xyz=0 0.010 -0.065 rpy=0 0 0; type continuous -> revolute
- joint lHipRoll: limit (none) -> lower=-0.52 upper=1.04 effort=40 velocity=25.0; origin xyz=0 0.0699999999999993 -0.0200000000000001 rpy=1.92592994438724E-34 0 0 -> xyz=0 0.07 -0.02 rpy=0 0 0; type continuous -> revolute
- joint lHipYaw: limit (none) -> lower=-1.04 upper=1.04 effort=40 velocity=25.0; origin xyz=-0.0222250000000002 0.0870035316828367 -0.29508 rpy=1.92592994438724E-34 0 0 -> xyz=-0.0222 0.0870 -0.2951 rpy=0 0 0; type continuous -> revolute
- joint lKnee: limit (none) -> lower=0.0 upper=2.13 effort=40 velocity=25.0; origin xyz=0 -0.016750000238715 -0.48 rpy=1.92592994438724E-34 0 0 -> xyz=0 -0.0168 -0.48 rpy=0 0 0; type continuous -> revolute
- joint rAnkle: limit (none) -> lower=0.901 upper=2.44 effort=40 velocity=25.0; origin xyz=0.0010775 -0.01675 -0.48 rpy=0 -1.57 0 -> xyz=0.0011 -0.0168 -0.48 rpy=0 -1.57 0; type continuous -> revolute
- joint rHipPitch: limit (none) -> lower=-1.04 upper=1.04 effort=40 velocity=25.0; origin xyz=0 -0.01 -0.065 rpy=1.9259E-34 0 0 -> xyz=0 -0.01 -0.065 rpy=0 0 0; type continuous -> revolute
- joint rHipRoll: limit (none) -> lower=-1.04 upper=0.52 effort=40 velocity=25.0; origin xyz=0 -0.07 -0.02 rpy=1.9259E-34 0 0 -> xyz=0 -0.07 -0.02 rpy=0 0 0; type continuous -> revolute
- joint rHipYaw: limit (none) -> lower=-1.04 upper=1.04 effort=40 velocity=25.0; origin xyz=-0.022225 -0.086996 -0.29508 rpy=1.9259E-34 0 0 -> xyz=-0.0222 -0.0870 -0.2951 rpy=0 0 0; type continuous -> revolute
- joint rKnee: limit (none) -> lower=0.0 upper=2.13 effort=40 velocity=25.0; type continuous -> revolute

Commit message: kinematic optimizer start

File: RobotSystem/RobotModel/Robot/Draco/Draco.urdf (robot description, URDF)
Before this commit: robot Draco, 17 links, 16 joints
Links:
- link torso: geometry 

Commit message: kinematics uniitest added

File: RobotSystem/RobotModel/Robot/Draco/Draco.urdf (robot description, URDF)
Before this commit: robot Draco, 17 links, 16 joints
Links:
- link torso: geometry visual mesh filename=meshes/torso.dae

Commit message: cent+kin test added

File: RobotSystem/RobotModel/Robot/Draco/Draco.urdf (robot description, URDF)
Before this commit: robot Draco, 17 links, 16 joints
Links:
- link torso: geometry visual mesh filename=meshes/torso_.dae

Commit message: sync

File: RobotSystem/RobotModel/Robot/Draco/Draco.urdf (robot description, URDF)
Before this commit: robot Draco, 17 links, 16 joints
Links:
- link lAnkle: mass 0.7 -> 0.4
- link rAnkle: mass 0.7 -> 0.4

File: RobotSystem/RobotModel/Robot/Draco/DracoFixed.urdf (robot description, URDF)
Before this commit: robot FixedDraco, 12 links, 11 joints
Links:
- link lAnkle: mass 0.7 -> 0.4
- link lHipPitch: mass 6.0 -> 5.5
- link lKnee: mass 3.5 -> 3.0
- link rAnkle: mass 0.7 -> 0.4

Commit message: tasks added

File: RobotSystem/RobotModel/Robot/Draco/Draco.urdf (robot description, URDF)
Before this commit: robot Draco, 17 links, 16 joints
Joints:
- joint lHipYaw: origin xyz=-0.0222 0.0870 -0.2951 rpy=0 0 0 -> xyz=-0.0222 0.0870 0.0 rpy=0 0 0
- joint rHipYaw: origin xyz=-0.0222 -0.0870 -0.2951 rpy=0 0 0 -> xyz=-0.0222 -0.0870 0.0 rpy=0 0 0

File: RobotSystem/RobotModel/Robot/Draco/DracoHanging.urdf (robot description, URDF)
Before this commit: robot Draco, 12 links, 11 joints
Links:
- added link basePosX, mass 0.00000001
- added link basePosY, mass 0.00000001
- added link basePosZ, mass 0.00000001
- added link baseRotY, mass 0.00000001
- added link baseRotZ, mass 0.00000001
- link lAnkle: mass 0.7 -> 0.4; geometry collision box size=0.15 0.04 0.03; visual mesh filename=meshes/lAnkle.dae
- link rAnkle: mass 0.7 -> 0.4
- link torso: geometry collision cylinder length=0.02 radius=0.1; visual mesh filename=meshes/torso_.dae
Joints:
- added joint basePosX: type prismatic, parent world, child basePosX, origin xyz=0 0 0 rpy=0 0 0, axis 1 0 0, limit lower=-200. upper=200. effort=100.0 velocity=100.0
- added joint basePosY: type prismatic, parent basePosX, child basePosY, origin xyz=0 0 0 rpy=0 0 0, axis 0 1 0, limit lower=-200. upper=200. effort=100.0 velocity=100.0
- added joint basePosZ: type prismatic, parent basePosY, child basePosZ, origin xyz=0 0 0 rpy=0 0 0, axis 0 0 1, limit lower=-200. upper=200. effort=100.0 velocity=100.0
- added joint baseRotY: type continuous, parent baseRotZ, child baseRotY, origin xyz=0 0 0 rpy=0 0 0, axis 0 1 0
- added joint baseRotZ: type continuous, parent basePosZ, child baseRotZ, origin xyz=0 0 0 rpy=0 0 0, axis 0 0 1
- joint baseRotX: axis (none) -> 1 0 0; parent world -> baseRotY; type floating -> continuous
- joint lAnkle: limit (none) -> lower=0.901 upper=2.44 effort=40 velocity=25.0; type continuous -> revolute
- joint lHipPitch: limit (none) -> lower=-1.04 upper=1.04 effort=40 velocity=25.0; type continuous -> revolute
- joint lHipRoll: limit (none) -> lower=-0.52 upper=1.04 effort=40 velocity=25.0; type continuous -> revolute
- joint lHipYaw: limit (none) -> lower=-1.04 upper=1.04 effort=40 velocity=25.0; origin xyz=-0.0222 0.0870 -0.2951 rpy=0 0 0 -> xyz=-0.0222 0.0870 0.0 rpy=0 0 0; type continuous -> revolute
- joint lKnee: limit (none) -> lower=0.0 upper=2.13 effort=40 velocity=25.0; type continuous -> revolute
- joint rAnkle: limit (none) -> lower=0.901 upper=2.44 effort=40 velocity=25.0; type continuous -> revolute
- joint rHipPitch: limit (none) -> lower=-1.04 upper=1.04 effort=40 velocity=25.0; type continuous -> revolute
- joint rHipRoll: limit (none) -> lower=-1.04 upper=0.52 effort=40 velocity=25.0; type continuous -> revolute
- joint rHipYaw: limit (none) -> lower=-1.04 upper=1.04 effort=40 velocity=25.0; origin xyz=-0.0222 -0.0870 -0.2951 rpy=0 0 0 -> xyz=-0.0222 -0.0870 0.0 rpy=0 0 0; type continuous -> revolute
- joint rKnee: limit (none) -> lower=0.0 upper=2.13 effort=40 velocity=25.0; type continuous -> revolute
