Commit message: walking parameters tuning

File: RobotSystem/RobotModel/Robot/Draco/DracoCollisionSim.urdf (robot description, URDF)
Before this commit: robot Draco, 26 links, 25 joints
Links:
- added link lFootBack2, mass 0.00001; collision sphere radius=0.03
- added link lFootFront2, mass 0.00001; collision sphere radius=0.03
- added link rFootBack2, mass 0.00001; collision sphere radius=0.03
- added link rFootFront2, mass 0.00001; collision sphere radius=0.03
Joints:
- added joint lFootBack2: type fixed, parent lAnkle, child lFootBack2, origin xyz=-0.05 -0.005 -0.044 rpy=0 0 0
- added joint lFootFront2: type fixed, parent lAnkle, child lFootFront2, origin xyz=0.08 -0.005 -0.044 rpy=0 0 0
- added joint rFootBack2: type fixed, parent rAnkle, child rFootBack2, origin xyz=-0.05 0.005 -0.044 rpy=0 0 0
- added joint rFootFront2: type fixed, parent rAnkle, child rFootFront2, origin xyz=0.08 0.005 -0.044 rpy=0 0 0
- joint lFootBack: origin xyz=-0.05 0 -0.044 rpy=0 0 0 -> xyz=-0.05 0.005 -0.044 rpy=0 0 0
- joint lFootFront: origin xyz=0.08 0 -0.044 rpy=0 0 0 -> xyz=0.08 0.005 -0.044 rpy=0 0 0
- joint rFootBack: origin xyz=-0.05 0 -0.044 rpy=0 0 0 -> xyz=-0.05 -0.005 -0.044 rpy=0 0 0
- joint rFootFront: origin xyz=0.08 0 -0.044 rpy=0 0 0 -> xyz=0.08 -0.005 -0.044 rpy=0 0 0
