Commit message: working_on_walking

File: RobotSystem/RobotModel/Robot/Draco/DracoCollision.urdf (robot description, URDF)
Before this commit: robot Draco, 21 links, 20 joints
Links:
- added link lFootCenter, mass 0.00001
- added link rFootCenter, mass 0.00001
Joints:
- added joint lFootCenter: type fixed, parent lAnkle, child lFootCenter, origin xyz=0.015 0 -0.059 rpy=0 0 0
- added joint rFootCenter: type fixed, parent rAnkle, child rFootCenter, origin xyz=0.015 0 -0.059 rpy=0 0 0

Commit message: before adding mocap at urdf

File: RobotSystem/RobotModel/Robot/Draco/DracoCollision.urdf (robot description, URDF)
Before this commit: robot Draco, 23 links, 22 joints
Joints:
- joint basePosX: limit lower=-200. upper=200. effort=100.0 velocity=100.0 -> lower=-200. upper=200. effort=150.0 velocity=100.0
- joint basePosY: limit lower=-200. upper=200. effort=100.0 velocity=100.0 -> lower=-200. upper=200. effort=150.0 velocity=100.0
- joint basePosZ: limit lower=-200. upper=200. effort=100.0 velocity=100.0 -> lower=-200. upper=200. effort=150.0 velocity=100.0
- joint lAnkle: limit lower=0.901 upper=2.44 effort=40 velocity=25.0 -> lower=0.901 upper=2.44 effort=150 velocity=25.0
- joint lHipPitch: limit lower=-1.04 upper=1.04 effort=40 velocity=25.0 -> lower=-1.04 upper=1.04 effort=150 velocity=25.0
- joint lHipRoll: limit lower=-0.52 upper=1.04 effort=40 velocity=25.0 -> lower=-0.52 upper=1.04 effort=150 velocity=25.0
- joint lHipYaw: limit lower=-1.04 upper=1.04 effort=40 velocity=25.0 -> lower=-1.04 upper=1.04 effort=150 velocity=25.0
- joint lKnee: limit lower=0.0 upper=2.13 effort=40 velocity=25.0 -> lower=0.0 upper=2.13 effort=150 velocity=25.0
- joint rAnkle: limit lower=0.901 upper=2.44 effort=40 velocity=25.0 -> lower=0.901 upper=2.44 effort=150 velocity=25.0
- joint rHipPitch: limit lower=-1.04 upper=1.04 effort=40 velocity=25.0 -> lower=-1.04 upper=1.04 effort=150 velocity=25.0
- joint rHipRoll: limit lower=-1.04 upper=0.52 effort=40 velocity=25.0 -> lower=-1.04 upper=0.52 effort=150 velocity=25.0
- joint rHipYaw: limit lower=-1.04 upper=1.04 effort=40 velocity=25.0 -> lower=-1.04 upper=1.04 effort=150 velocity=25.0
- joint rKnee: limit lower=0.0 upper=2.13 effort=40 velocity=25.0 -> lower=0.0 upper=2.13 effort=150 velocity=25.0

Commit message: body_led_added_in_urdf

File: RobotSystem/RobotModel/Robot/Draco/DracoCollision.urdf (robot description, URDF)
Before this commit: robot Draco, 23 links, 22 joints
Links:
- added link led_torso_center, mass 0.00001
- added link led_torso_left, mass 0.00001
- added link led_torso_right, mass 0.00001
Joints:
- added joint led_torso_center: type fixed, parent torso, child led_torso_center, origin xyz=0.077 0 0 rpy=0 0 0
- added joint led_torso_left: type fixed, parent torso, child led_torso_left, origin xyz=0.077 0.0405 -0.0175 rpy=0 0 0
- added joint led_torso_right: type fixed, parent torso, child led_torso_right, origin xyz=0.077 -0.0405 -0.0175 rpy=0 0 0

Commit message: body ori estimator added but needed to be validated && led pos announcer added

File: RobotSystem/RobotModel/Robot/Draco/DracoCollision.urdf (robot description, URDF)
Before this commit: robot Draco, 26 links, 25 joints
Links:
- removed link led_torso_center
- removed link led_torso_left
- removed link led_torso_right
- removed link torso
- added link Torso, mass 9.67; collision cylinder length=0.02 radius=0.1; visual mesh filename=meshes/torso_.dae
- added link cTorsoLed, mass 0.00001
- added link lTorsoLed, mass 0.00001
- added link rTorsoLed, mass 0.00001
Joints:
- removed joint led_torso_center
- removed joint led_torso_left
- removed joint led_torso_right
- added joint cTorsoLed: type fixed, parent Torso, child cTorsoLed, origin xyz=0.077 0 0 rpy=0 0 0
- added joint lTorsoLed: type fixed, parent Torso, child lTorsoLed, origin xyz=0.077 0.0405 -0.0175 rpy=0 0 0
- added joint rTorsoLed: type fixed, parent Torso, child rTorsoLed, origin xyz=0.077 -0.0405 -0.0175 rpy=0 0 0
- joint baseRotX: child torso -> Torso
- joint lHipYaw: parent torso -> Torso
- joint rHipYaw: parent torso -> Torso

File: RobotSystem/RobotModel/Robot/Draco/DracoCollisionSim.urdf (robot description, URDF)
Before this commit: robot Draco, 30 links, 29 joints
Links:
- removed link led_torso_center
- removed link led_torso_left
- removed link led_torso_right
- removed link torso
- added link Torso, mass 9.67; collision cylinder length=0.02 radius=0.1; visual mesh filename=meshes/torso_.dae
- added link cTorsoLed, mass 0.00001
- added link lTorsoLed, mass 0.00001
- added link rTorsoLed, mass 0.00001
Joints:
- removed joint led_torso_center
- removed joint led_torso_left
- removed joint led_torso_right
- added joint cTorsoLed: type fixed, parent Torso, child cTorsoLed, origin xyz=0.077 0 0 rpy=0 0 0
- added joint lTorsoLed: type fixed, parent Torso, child lTorsoLed, origin xyz=0.077 0.0405 -0.0175 rpy=0 0 0
- added joint rTorsoLed: type fixed, parent Torso, child rTorsoLed, origin xyz=0.077 -0.0405 -0.0175 rpy=0 0 0
- joint baseRotX: child torso -> Torso
- joint lHipYaw: parent torso -> Torso
- joint rHipYaw: parent torso -> Torso

Commit message: before working on sim

File: RobotSystem/RobotModel/Robot/Draco/DracoCollision.urdf (robot description, URDF)
Before this commit: robot Draco, 26 links, 25 joints
Joints:
- joint lFootCenter: origin xyz=0.015 0 -0.059 rpy=0 0 0 -> xyz=0.026 0.0168 -0.48 rpy=0 0 0; parent lAnkle -> lKnee
- joint rFootCenter: origin xyz=0.015 0 -0.059 rpy=0 0 0 -> xyz=0.026 -0.0168 -0.48 rpy=0 0 0; parent rAnkle -> rKnee

Commit message: before testing params

File: RobotSystem/RobotModel/Robot/Draco/DracoCollision.urdf (robot description, URDF)
Before this commit: robot Draco, 26 links, 25 joints
Joints:
- joint cTorsoLed: origin xyz=0.077 0 0 rpy=0 0 0 -> xyz=0.077 0 0.05 rpy=0 0 0
- joint lFootCenter: origin xyz=0.026 0.0168 -0.48 rpy=0 0 0 -> xyz=0.02 0 -0.059 rpy=0 0 0; parent lKnee -> lAnkle
- joint lTorsoLed: origin xyz=0.077 0.0405 -0.0175 rpy=0 0 0 -> xyz=0.077 0.0405 0.25 rpy=0 0 0
- joint rFootCenter: origin xyz=0.026 -0.0168 -0.48 rpy=0 0 0 -> xyz=0.02 0 -0.059 rpy=0 0 0; parent rKnee -> rAnkle
- joint rTorsoLed: origin xyz=0.077 -0.0405 -0.0175 rpy=0 0 0 -> xyz=0.077 -0.0405 0.25 rpy=0 0 0

File: RobotSystem/RobotModel/Robot/Draco/DracoCollisionSim.urdf (robot description, URDF)
Before this commit: robot Draco, 30 links, 29 joints
Joints:
- joint cTorsoLed: origin xyz=0.077 0 0 rpy=0 0 0 -> xyz=0.077 0 0.05 rpy=0 0 0
- joint lTorsoLed: origin xyz=0.077 0.0405 -0.0175 rpy=0 0 0 -> xyz=0.077 0.0405 0.25 rpy=0 0 0
- joint rTorsoLed: origin xyz=0.077 -0.0405 -0.0175 rpy=0 0 0 -> xyz=0.077 -0.0405 0.25 rpy=0 0 0

Commit message: walking

File: RobotSystem/RobotModel/Robot/Draco/DracoCollision.urdf (robot description, URDF)
Before this commit: robot Draco, 26 links, 25 joints
Links:
- link Torso: mass 9.67 -> 10.0
- link lHipPitch: mass 6.0 -> 9.0
- link rHipPitch: mass 6.0 -> 9.0
Joints:
- joint lFootCenter: origin xyz=0.02 0 -0.059 rpy=0 0 0 -> xyz=0 0 -0.03 rpy=0 0 0
- joint rFootCenter: origin xyz=0.02 0 -0.059 rpy=0 0 0 -> xyz=0 0 -0.03 rpy=0 0 0
