Commit message: cart pole system is added for reinforcement learning

File: RobotSystem/RobotModel/Robot/CartPole/CartPole.urdf (robot description, URDF)
Before this commit: robot cart_pole, 4 links, 3 joints
Links:
- link slideBar: mass 0 -> 1.0

Commit message: data generating part

File: RobotSystem/RobotModel/Robot/CartPole/CartPole.urdf (robot description, URDF)
Before this commit: robot cart_pole, 4 links, 3 joints
Links:
- link pole: mass 10 -> 0.1

Commit message: move servo_rate and ip_address to definition file

File: RobotSystem/RobotModel/Robot/CartPole/CartPole.urdf (robot description, URDF)
Before this commit: robot cart_pole, 4 links, 3 joints
Links:
- link pole: mass 0.1 -> 0.3
