Commit message: better draco visualization

File: RobotSystem/RobotModel/Ground/ground_terrain.urdf (robot description, URDF)
Before this commit: robot ground_skeleton, 2 links, 1 joints
Links:
- link ground_link: geometry collision box size=5.0 5.0 0.05; visual mesh filename=tile_marble_diamond.dae scale=1. 1. 1.

File: RobotSystem/RobotModel/Robot/Draco/Draco.urdf (robot description, URDF)
Before this commit: robot Draco, 12 links, 11 joints
Links:
- link lAnkle: geometry collision mesh filename=meshes/lAnkle.dae; visual mesh filename=meshes/lAnkle.dae
- link lHipPitch: geometry visual mesh filename=meshes/lHipPitch.dae
- link lHipRoll: geometry visual mesh filename=meshes/lHipRoll.dae
- link lHipYaw: geometry visual mesh filename=meshes/lHipYaw.dae
- link lKnee: geometry visual mesh filename=meshes/lKnee.dae
- link rAnkle: geometry collision mesh filename=meshes/rAnkle.dae; visual mesh filename=meshes/rAnkle.dae
- link rHipPitch: geometry visual mesh filename=meshes/rHipPitch.dae
- link rHipRoll: geometry visual mesh filename=meshes/rHipRoll.dae
- link rHipYaw: geometry visual mesh filename=meshes/rHipYaw.dae
- link rKnee: geometry visual mesh filename=meshes/rKnee.dae
- link torso: geometry visual mesh filename=meshes/torso.dae

Commit message: under finding parameters for walking forward

File: RobotSystem/RobotModel/Ground/ground_terrain.urdf (robot description, URDF)
Before this commit: robot ground_skeleton, 2 links, 1 joints
Links:
- link ground_link: geometry collision box size=50.0 50.0 0.05; visual mesh filename=tile_marble_diamond.dae scale=1. 1. 1.
