Commit message: pybullet draco model is added

File: RobotModel/Robot/Draco/DracoFixed.urdf (robot description, URDF)
Before this commit: robot FixedDraco, 12 links, 11 joints
Links:
- removed link torso
- removed link world
- added link Torso, mass 9.67; collision cylinder length=0.02 radius=0.1; visual mesh filename=meshes/torso_.dae
- added link cTorsoLed, mass 0.00001
- added link lFootBack, mass 0.00001; collision sphere radius=0.03
- added link lFootBack2, mass 0.00001; collision sphere radius=0.03
- added link lFootCenter, mass 0.00001
- added link lFootFront, mass 0.00001; collision sphere radius=0.03
- added link lFootFront2, mass 0.00001; collision sphere radius=0.03
- added link lTorsoLed, mass 0.00001
- added link rFootBack, mass 0.00001; collision sphere radius=0.03
- added link rFootBack2, mass 0.00001; collision sphere radius=0.03
- added link rFootCenter, mass 0.00001
- added link rFootFront, mass 0.00001; collision sphere radius=0.03
- added link rFootFront2, mass 0.00001; collision sphere radius=0.03
- added link rTorsoLed, mass 0.00001
- link lAnkle: geometry visual mesh filename=meshes/lAnkle.dae
- link lHipPitch: mass 5.0 -> 6.0
- link lKnee: mass 3.1 -> 3.5
- link rAnkle: geometry visual mesh filename=meshes/rAnkle.dae
- link rHipPitch: mass 5.0 -> 6.0
- link rKnee: mass 3.1 -> 3.5
Joints:
- removed joint torso
- added joint cTorsoLed: type fixed, parent Torso, child cTorsoLed, origin xyz=0.077 0 0.05 rpy=0 0 0
- added joint lFootBack: type fixed, parent lAnkle, child lFootBack, origin xyz=-0.05 0.005 -0.044 rpy=0 0 0
- added joint lFootBack2: type fixed, parent lAnkle, child lFootBack2, origin xyz=-0.05 -0.005 -0.044 rpy=0 0 0
- added joint lFootCenter: type fixed, parent lAnkle, child lFootCenter, origin xyz=0.015 0 -0.059 rpy=0 0 0
- added joint lFootFront: type fixed, parent lAnkle, child lFootFront, origin xyz=0.08 0.005 -0.044 rpy=0 0 0
- added joint lFootFront2: type fixed, parent lAnkle, child lFootFront2, origin xyz=0.08 -0.005 -0.044 rpy=0 0 0
- added joint lTorsoLed: type fixed, parent Torso, child lTorsoLed, origin xyz=0.077 0.0405 0.25 rpy=0 0 0
- added joint rFootBack: type fixed, parent rAnkle, child rFootBack, origin xyz=-0.05 -0.005 -0.044 rpy=0 0 0
- added joint rFootBack2: type fixed, parent rAnkle, child rFootBack2, origin xyz=-0.05 0.005 -0.044 rpy=0 0 0
- added joint rFootCenter: type fixed, parent rAnkle, child rFootCenter, origin xyz=0.015 0 -0.059 rpy=0 0 0
- added joint rFootFront: type fixed, parent rAnkle, child rFootFront, origin xyz=0.08 -0.005 -0.044 rpy=0 0 0
- added joint rFootFront2: type fixed, parent rAnkle, child rFootFront2, origin xyz=0.08 0.005 -0.044 rpy=0 0 0
- added joint rTorsoLed: type fixed, parent Torso, child rTorsoLed, origin xyz=0.077 -0.0405 0.25 rpy=0 0 0
- joint lAnkle: limit (none) -> lower=0.901 upper=2.44 effort=150 velocity=25.0; type continuous -> revolute
- joint lHipPitch: limit (none) -> lower=-1.04 upper=1.04 effort=150 velocity=25.0; type continuous -> revolute
- joint lHipRoll: limit (none) -> lower=-0.52 upper=1.04 effort=150 velocity=25.0; type continuous -> revolute
- joint lHipYaw: limit (none) -> lower=-1.04 upper=1.04 effort=150 velocity=25.0; origin xyz=-0.0222 0.0870 -0.2951 rpy=0 0 0 -> xyz=-0.0222 0.0870 0.0 rpy=0 0 0; parent torso -> Torso; type continuous -> revolute
- joint lKnee: limit (none) -> lower=0.0 upper=2.13 effort=150 velocity=25.0; type continuous -> revolute
- joint rAnkle: limit (none) -> lower=0.901 upper=2.44 effort=150 velocity=25.0; type continuous -> revolute
- joint rHipPitch: limit (none) -> lower=-1.04 upper=1.04 effort=150 velocity=25.0; type continuous -> revolute
- joint rHipRoll: limit (none) -> lower=-1.04 upper=0.52 effort=150 velocity=25.0; type continuous -> revolute
- joint rHipYaw: limit (none) -> lower=-1.04 upper=1.04 effort=150 velocity=25.0; origin xyz=-0.0222 -0.0870 -0.2951 rpy=0 0 0 -> xyz=-0.0222 -0.0870 0.0 rpy=0 0 0; parent torso -> Torso; type continuous -> revolute
- joint rKnee: limit (none) -> lower=0.0 upper=2.13 effort=150 velocity=25.0; type continuous -> revolute
