Commit message: updated .gitattribute

File: RobotModel/Robot/Valkyrie/materials/materials.xacro (robot description, xacro)
@@ -1,15 +1,3 @@
-<?xml version="1.0" ?>
-<robot xmlns:xacro="http://www.ros.org/wiki/xacro" name="v1/materials">
-    <material name="White">
-        <color rgba="1.0 1.0 1.0 1.0"/>
-    </material>
-    <material name="Gold">
-        <color rgba="1.0 0.67 0 1.0"/>
-    </material>
-    <material name="Gray">
-        <color rgba="0.5 0.5 0.5 1.0"/>
-    </material>
-    <material name="Pink">
-        <color rgba="0.8 0 0.45 1.0"/>
-    </material>
-</robot>
+version https://git-lfs.github.com/spec/v1
+oid sha256:9fdebadf253e44e3a2932961f722b3872d991dfb49286413339a0d1590fbe633
+size 441
