Commit message: now dealing with segfault

File: RobotModel/ground/plane.urdf (robot description, URDF)
Before this commit: robot plane, 1 links, 0 joints
Links:
- link planeLink: mass .0 -> 0.001; geometry visual mesh filename=plane.obj scale=1 1 1

Commit message: before converting qd to v4

File: RobotModel/ground/plane.urdf (robot description, URDF)
Before this commit: robot plane, 1 links, 0 joints
Links:
- link planeLink: geometry collision plane normal=0 0 1; visual mesh filename=plane.obj scale=1 1 1
