Commit message: incorporate new urdf, need to figure out what would be the right value for knee_adj_param for draco.urdf

File: RobotModel/draco/draco.urdf (robot description, URDF)
Before this commit: robot draco_3, 39 links, 38 joints
Links:
- added link torso_imu, mass 1e-9
- link l_ankle_fe_link: mass 0.183143 -> 0.172
- link l_ankle_ie_link: mass 0.436553 -> 0.478
- link l_elbow_fe_link: mass 0.989887 -> 0.990031
- link l_hip_aa_link: mass 0.77975 -> 0.912
- link l_hip_fe_link: mass 4.549 -> 5.0
- link l_hip_ie_link: mass 0.139743 -> 0.162
- link l_knee_adj_link: mass 0.090042 -> 0.156
- link l_knee_fe_ld: mass 2.55664 -> 2.5
- link l_knee_fe_lp: mass 0.135683 -> 0.211
- link l_sake_gripper_link: mass 0.545 -> 0.498
- link neck_pitch_link: mass 1.22948 -> 1.394979
- link r_ankle_fe_link: mass 0.183145 -> 0.172
- link r_ankle_ie_link: mass 0.437539 -> 0.478
- link r_hip_aa_link: mass 0.849423 -> 0.912
- link r_hip_fe_link: mass 4.983 -> 5.0
- link r_hip_ie_link: mass 0.139506 -> 0.162
- link r_knee_adj_link: mass 0.090042 -> 0.156
- link r_knee_fe_ld: mass 2.58619 -> 2.5
- link r_knee_fe_lp: mass 0.152083 -> 0.211
- link r_sake_gripper_link: mass 0.545 -> 0.498
- link torso_link: mass 6.41443 -> 6.456
Joints:
- added joint torso_imu_frame: type fixed, parent torso_link, child torso_imu, origin xyz=0 0 -0.09 rpy=3.14159 0 3.14159, axis 0 0 0
- joint l_elbow_fe: limit lower=-2.0944 upper=0.0872665 effort=10 velocity=37.1 -> lower=-2.094 upper=0.0872665 effort=10 velocity=59.2
- joint l_knee_fe_jd: origin xyz=0 0 -0.1115386 rpy=0 0 0 -> xyz=0.0 0.0 -0.1117386 rpy=0 0 0
- joint l_shoulder_aa: limit lower=0 upper=2.0944 effort=18 velocity=30 -> lower=0 upper=2.0944 effort=18 velocity=47
- joint l_shoulder_fe: limit lower=-2.26893 upper=0.698132 effort=18 velocity=30 -> lower=-2.26893 upper=0.698132 effort=18 velocity=47
- joint l_shoulder_ie: limit lower=-1.48353 upper=1.48353 effort=18 velocity=30 -> lower=-1.55 upper=1.55 effort=18 velocity=47
- joint l_wrist_pitch: limit lower=-1.5708 upper=1.5708 effort=8.8 velocity=82.8 -> lower=-1.571 upper=1.571 effort=8.8 velocity=76
- joint l_wrist_ps: limit lower=-1.5708 upper=1.5708 effort=12 velocity=44.5 -> lower=-1.571 upper=1.571 effort=12 velocity=71
- joint neck_pitch: limit lower=-0.523599 upper=1.309 effort=8.8 velocity=82.8 -> lower=-0.523599 upper=1.309 effort=8.8 velocity=76
- joint r_elbow_fe: limit lower=-2.0944 upper=0.0872665 effort=10 velocity=37.1 -> lower=-2.094 upper=0.0872665 effort=10 velocity=59.2
- joint r_knee_fe_jd: origin xyz=0 0 -0.1115386 rpy=0 0 0 -> xyz=0 0 -0.1117386 rpy=0 0 0
- joint r_shoulder_aa: limit lower=-2.0944 upper=0 effort=18 velocity=30 -> lower=-2.0944 upper=0 effort=18 velocity=47
- joint r_shoulder_fe: limit lower=-2.26893 upper=0.698132 effort=18 velocity=30 -> lower=-2.26893 upper=0.698132 effort=18 velocity=47
- joint r_shoulder_ie: limit lower=-1.48353 upper=1.48353 effort=18 velocity=30 -> lower=-1.5 upper=1.5 effort=18 velocity=47
- joint r_wrist_pitch: limit lower=-1.5708 upper=1.5708 effort=8.8 velocity=82.8 -> lower=-1.571 upper=1.571 effort=8.8 velocity=76
- joint r_wrist_ps: limit lower=-1.5708 upper=1.5708 effort=12 velocity=44.5 -> lower=-1.571 upper=1.571 effort=12 velocity=71
- joint torso_com: origin xyz=-0.0310745 -0.000497416 0.137484 rpy=0 0 0 -> xyz=-31.658e-03 -0.03865e-03 125.19e-03 rpy=0 0 0

File: RobotModel/draco/draco_apptronik_sim.urdf (robot description, URDF)
Before this commit: robot draco, 40 links, 39 joints
Links:
- link l_ankle_fe_link: geometry visual mesh filename=package://meshes/l_ankle_fe_link.stl
- link l_ankle_ie_link: geometry collision box size=0.2 0.1 0.0591; visual mesh filename=package://meshes/l_ankle_ie_link.stl
- link l_elbow_fe_link: geometry visual mesh filename=package://meshes/l_elbow_fe_link.stl
- link l_hip_aa_link: geometry visual mesh filename=package://meshes/l_hip_aa_link.stl
- link l_hip_fe_link: geometry visual mesh filename=package://meshes/l_hip_fe_link.stl
- link l_hip_ie_link: geometry visual mesh filename=package://meshes/l_hip_ie_link.stl
- link l_knee_adj_link: geometry visual mesh filename=package://meshes/l_knee_adj_link.stl
- link l_knee_fe_ld: geometry visual mesh filename=package://meshes/l_knee_fe_ld.stl
- link l_knee_fe_lp: geometry visual mesh filename=package://meshes/l_knee_fe_lp.stl
- link l_sake_gripper_link: geometry visual mesh filename=package://meshes/l_sake_gripper_link.stl
- link l_shoulder_aa_link: geometry visual mesh filename=package://meshes/l_shoulder_aa_link.stl
- link l_shoulder_fe_link: geometry visual mesh filename=package://meshes/l_shoulder_fe_link.stl
- link l_shoulder_ie_link: geometry visual mesh filename=package://meshes/l_shoulder_ie_link.stl
- link l_wrist_ps_link: geometry visual mesh filename=package://meshes/l_wrist_ps_link.stl
- link neck_pitch_link: geometry visual mesh filename=package://meshes/neck_pitch_link.stl
- link r_ankle_fe_link: geometry visual mesh filename=package://meshes/r_ankle_fe_link.stl
- link r_ankle_ie_link: geometry collision box size=0.2 0.1 0.0591; visual mesh filename=package://meshes/r_ankle_ie_link.stl
- link r_elbow_fe_link: geometry visual mesh filename=package://meshes/r_elbow_fe_link.stl
- link r_hip_aa_link: geometry visual mesh filename=package://meshes/r_hip_aa_link.stl
- link r_hip_fe_link: geometry visual mesh filename=package://meshes/r_hip_fe_link.stl
- link r_hip_ie_link: geometry visual mesh filename=package://meshes/r_hip_ie_link.stl
- link r_knee_adj_link: geometry visual mesh filename=package://meshes/r_knee_adj_link.stl
- link r_knee_fe_ld: geometry visual mesh filename=package://meshes/r_knee_fe_ld.stl
- link r_knee_fe_lp: geometry visual mesh filename=package://meshes/r_knee_fe_lp.stl
- link r_sake_gripper_link: geometry visual mesh filename=package://meshes/r_sake_gripper_link.stl
- link r_shoulder_aa_link: geometry visual mesh filename=package://meshes/r_shoulder_aa_link.stl
- link r_shoulder_fe_link: geometry visual mesh filename=package://meshes/r_shoulder_fe_link.stl
- link r_shoulder_ie_link: geometry visual mesh filename=package://meshes/r_shoulder_ie_link.stl
- link r_wrist_ps_link: geometry visual mesh filename=package://meshes/r_wrist_ps_link.stl
- link torso_link: geometry visual mesh filename=package://meshes/torso_link.stl
