Commit message: draco torso & neck mesh file updated with .obj file format

File: robot_model/draco/draco.urdf (robot description, URDF)
Before this commit: robot draco, 40 links, 39 joints
Links:
- link neck_pitch_link: geometry visual mesh filename=package://meshes/neck_pitch_link.obj
- link torso_link: geometry visual mesh filename=package://meshes/torso_link.obj

Commit message: added extra frames around the feet for mpc

File: robot_model/draco/draco.urdf (robot description, URDF)
Before this commit: robot draco, 40 links, 39 joints
Links:
- added link base_link
- added link l_foot_contact_lower_left
- added link l_foot_contact_lower_right
- added link l_foot_contact_upper_left
- added link l_foot_contact_upper_right
- added link r_foot_contact_lower_left
- added link r_foot_contact_lower_right
- added link r_foot_contact_upper_left
- added link r_foot_contact_upper_right
- added link world
Joints:
- added joint base_joint: type floating, parent world, child base_link
- added joint base_torso_joint: type fixed, parent base_link, child torso_link
- added joint l_foot_contact_frame_lower_left: type fixed, parent l_foot_contact, child l_foot_contact_lower_left, origin xyz=-0.1 0.05 0.0 rpy=0 0 0
- added joint l_foot_contact_frame_lower_right: type fixed, parent l_foot_contact, child l_foot_contact_lower_right, origin xyz=-0.1 -0.05 0.0 rpy=0 0 0
- added joint l_foot_contact_frame_upper_left: type fixed, parent l_foot_contact, child l_foot_contact_upper_left, origin xyz=0.1 0.05 0.0 rpy=0 0 0
- added joint l_foot_contact_frame_upper_right: type fixed, parent l_foot_contact, child l_foot_contact_upper_right, origin xyz=0.1 -0.05 0.0 rpy=0 0 0
- added joint r_foot_contact_frame_lower_left: type fixed, parent r_foot_contact, child r_foot_contact_lower_left, origin xyz=-0.1 0.05 0.0 rpy=0 0 0
- added joint r_foot_contact_frame_lower_right: type fixed, parent r_foot_contact, child r_foot_contact_lower_right, origin xyz=-0.1 -0.05 0.0 rpy=0 0 0
- added joint r_foot_contact_frame_upper_left: type fixed, parent r_foot_contact, child r_foot_contact_upper_left, origin xyz=0.1 0.05 0.0 rpy=0 0 0
- added joint r_foot_contact_frame_upper_right: type fixed, parent r_foot_contact, child r_foot_contact_upper_right, origin xyz=0.1 -0.05 0.0 rpy=0 0 0

File: robot_model/draco3/draco3_gripper_mesh_updated.urdf (robot description, URDF)
Before this commit: robot draco_3, 49 links, 48 joints
Links:
- added link l_foot_contact_lower_left
- added link l_foot_contact_lower_right
- added link l_foot_contact_upper_left
- added link l_foot_contact_upper_right
- added link r_foot_contact_lower_left
- added link r_foot_contact_lower_right
- added link r_foot_contact_upper_left
- added link r_foot_contact_upper_right
Joints:
- added joint l_foot_contact_frame_lower_left: type fixed, parent l_foot_contact, child l_foot_contact_lower_left, origin xyz=-0.1 0.05 0.0 rpy=0 0 0
- added joint l_foot_contact_frame_lower_right: type fixed, parent l_foot_contact, child l_foot_contact_lower_right, origin xyz=-0.1 -0.05 0.0 rpy=0 0 0
- added joint l_foot_contact_frame_upper_left: type fixed, parent l_foot_contact, child l_foot_contact_upper_left, origin xyz=0.1 0.05 0.0 rpy=0 0 0
- added joint l_foot_contact_frame_upper_right: type fixed, parent l_foot_contact, child l_foot_contact_upper_right, origin xyz=0.1 -0.05 0.0 rpy=0 0 0
- added joint r_foot_contact_frame_lower_left: type fixed, parent r_foot_contact, child r_foot_contact_lower_left, origin xyz=-0.1 0.05 0.0 rpy=0 0 0
- added joint r_foot_contact_frame_lower_right: type fixed, parent r_foot_contact, child r_foot_contact_lower_right, origin xyz=-0.1 -0.05 0.0 rpy=0 0 0
- added joint r_foot_contact_frame_upper_left: type fixed, parent r_foot_contact, child r_foot_contact_upper_left, origin xyz=0.1 0.05 0.0 rpy=0 0 0
- added joint r_foot_contact_frame_upper_right: type fixed, parent r_foot_contact, child r_foot_contact_upper_right, origin xyz=0.1 -0.05 0.0 rpy=0 0 0

Commit message: added base_joint offset

File: robot_model/draco/draco.urdf (robot description, URDF)
Before this commit: robot draco, 50 links, 49 joints
Joints:
- joint base_joint: origin (none) -> xyz=-0.05 -0.1 0.742691 rpy=0 0 0

Commit message: commit

File: robot_model/draco/draco.urdf (robot description, URDF)
Before this commit: robot draco, 50 links, 49 joints
Links:
- link l_foot_contact_lower_left: mass None -> 1e-9
- link l_foot_contact_lower_right: mass None -> 1e-9
- link l_foot_contact_upper_left: mass None -> 1e-9
- link l_foot_contact_upper_right: mass None -> 1e-9
- link r_foot_contact_lower_left: mass None -> 1e-9
- link r_foot_contact_lower_right: mass None -> 1e-9
- link r_foot_contact_upper_left: mass None -> 1e-9
- link r_foot_contact_upper_right: mass None -> 1e-9
