Commit message: comparing with pypnc

File: robot_model/draco/draco_rel_path.urdf (robot description, URDF)
Before this commit: robot draco, 40 links, 39 joints
Links:
- added link world
Joints:
- added joint world_to_torso: type fixed, parent world, child torso_link, origin xyz=0 0 0 rpy=0 0 0

Commit message: draco hand reaching task testing done

File: robot_model/draco/draco_rel_path.urdf (robot description, URDF)
Before this commit: robot draco, 40 links, 39 joints
Links:
- link torso_link: mass 7.856 -> 6.456

Commit message: added visualization of bigger feet and respective STLs
still need to add foot mass difference

File: robot_model/draco/draco_rel_path.urdf (robot description, URDF)
Before this commit: robot draco, 40 links, 39 joints
Links:
- link l_ankle_ie_link: geometry collision box size=0.2 0.1 0.0591; visual mesh filename=meshes/l_ankle_ie_link_big_foot.stl
- link r_ankle_ie_link: geometry collision box size=0.2 0.1 0.0591; visual mesh filename=meshes/r_ankle_ie_link_big_foot.stl

File: robot_model/draco3/draco3_gripper_mesh_updated.urdf (robot description, URDF)
Before this commit: robot draco_3, 49 links, 48 joints
Links:
- link l_ankle_ie_link: geometry collision box size=0.25 0.15 0.0591; visual mesh filename=package://meshes/l_ankle_ie_link_big_foot.stl
- link r_ankle_ie_link: geometry collision box size=0.25 0.15 0.0591; visual mesh filename=package://meshes/r_ankle_ie_link_big_foot.stl

Commit message: match collision box in feet to bigger feet and updated visuals

File: robot_model/draco/draco_rel_path.urdf (robot description, URDF)
Before this commit: robot draco, 40 links, 39 joints
Links:
- link l_ankle_ie_link: geometry collision box size=0.25 0.15 0.0591; visual mesh filename=meshes/l_ankle_ie_link_big_foot.stl
- link r_ankle_ie_link: geometry collision box size=0.25 0.15 0.0591; visual mesh filename=meshes/r_ankle_ie_link_big_foot.stl
